Commit message: Added world and model changes

File: gym_gazebo/envs/installation/catkin_ws/src/snakemonster/snake_monster/urdf/my_snake_monster.xacro (robot description, xacro)
@@ -150,32 +150,4 @@
     <origin xyz="${-width/2} -${leg_y_offset} ${height/2}" rpy="-${PI/2} 0 ${PI/2}"/>
   </joint>
-    <xacro:property name="camera_link" value="0.05" /> <!-- Size of square 'camera' box -->
-    <joint name="camera_joint" type="fixed">
-    <axis xyz="0 1 0" />
-    <origin xyz="0 0.125 0.052" rpy="0 0 1.57"/>
-    <parent link="base"/>
-    <child link="camera_link"/>
-  </joint>
-  <!-- Camera -->
-  <link name="camera_link">
-    <collision>
-      <origin xyz="0 0 0.052" rpy="0 0 1.57"/>
-      <geometry>
-    <box size="${camera_link} ${camera_link} ${camera_link}"/>
-      </geometry>
-    </collision>
-    <visual>
-      <origin xyz="-0.02 -0.02 0.024" rpy="0 0 0"/>
-      <geometry>
-    <mesh filename="package://snake_monster/meshes/gopro.dae"/>
-      </geometry>
-      <material name="red"/>
-    </visual>
-    <inertial>
-      <mass value="1e-5" />
-      <origin xyz="0 0 0" rpy="0 0 0"/>
-      <inertia ixx="1e-6" ixy="0" ixz="0" iyy="1e-6" iyz="0" izz="1e-6" />
-    </inertial>
-  </link>
  <xacro:include filename="$(find kobuki_description)/urdf/sensors/lidar_sensor.urdf.xacro" />
  <xacro:lidar_sensor
@@ -195,4 +167,33 @@
   <!-- Import all Gazebo-customization elements -->
   <xacro:include filename="./my_snake_monster.gazebo" />
+<xacro:property name="camera_link" value="0.05"/><!-- Size of square 'camera' box --><joint name="camera_joint" type="fixed"><axis xyz="0 1 0"/><origin xyz="0 0.125 0.052" rpy="0 0 1.57"/><parent link="base"/><child link="camera_link"/></joint><!-- Camera --><link name="camera_link"><collision><origin xyz="0 0 0.052" rpy="0 0 1.57"/><geometry><box size="${camera_link} ${camera_link} ${camera_link}"/></geometry></collision><visual><origin xyz="-0.02 -0.02 0.024" rpy="0 0 0"/><geometry><mesh filename="package://snake_monster/meshes/gopro.dae"/></geometry><material name="red"/></visual><inertial><mass value="1e-5"/><origin xyz="0 0 0" rpy="0 0 0"/><inertia ixx="1e-6" ixy="0" ixz="0" iyy="1e-6" iyz="0" izz="1e-6"/></inertial></link>
+   <xacro:property name="imu_link" value="0.05" /> <!-- Size of square 'camera' box -->
+    <joint name="imu_joint" type="fixed">
+    <axis xyz="0 1 0" />
+    <origin xyz="0 0.125 0.052" rpy="0 0 1.57"/>
+    <parent link="base"/>
+    <child link="imu_link"/>
+  </joint>
+  <!-- IMU -->
+  <link name="imu_link">
+    <collision>
+      <origin xyz="0 0 0.052" rpy="0 0 1.57"/>
+      <geometry>
+    <box size="0.1 0.1 0.1"/>
+      </geometry>
+    </collision>
+    <visual>
+      <origin xyz="-0.02 -0.02 0.024" rpy="0 0 0"/>
+      <geometry>
+    <box size ="0.1 0.1 0.1"/>
+      </geometry>
+      <material name="red"/>
+    </visual>
+    <inertial>
+      <mass value="1e-5" />
+      <origin xyz="0 0 0" rpy="0 0 0"/>
+      <inertia ixx="1e-6" ixy="0" ixz="0" iyy="1e-6" iyz="0" izz="1e-6" />
+    </inertial>
+  </link>
   <!-- legs -->
   <xacro:leg leg="leg1" mod1="${L1_1}" mod2="${L1_2}" mod3="${L1_3}"/>

Commit message: A few state additions and reqard calculations for Flavian's headstart

File: gym_gazebo/envs/installation/catkin_ws/src/snakemonster/snake_monster/urdf/my_snake_monster.xacro (robot description, xacro)
@@ -1,62 +1,62 @@
 <?xml version="1.0"?>
 <robot xmlns:xacro="http://www.ros.org/wiki/xacro" name="snake_monster">
-  <!-- *************************** XACRO MACROS *************************** -->
-  <xacro:property name="PI" value="3.1415926535897931" />
-  <xacro:property name="M_PI" value="3.141592653589793" />
-  <!-- load macros for modules -->
-  <xacro:include filename="./module_common.xacro"/>
-  <xacro:include filename="./rotary_module.xacro"/>
-  <xacro:include filename="./extension_module.xacro"/>
-  <xacro:include filename="./elbow_module_snake_monster.xacro"/>
-  <xacro:include filename="./leg.xacro"/>
-  <!-- ************************* ROBOT DEFINITION ************************* -->
-  <xacro:property name="L1_1" value="SA014__MoJo" />
-  <xacro:property name="L1_2" value="SA013__MoJo" />
-  <xacro:property name="L1_3" value="SA023__MoJo" />
-  <xacro:property name="L2_1" value="SA037__MoJo" />
-  <xacro:property name="L2_2" value="SA049__MoJo" />
-  <xacro:property name="L2_3" value="SA030__MoJo" />
-  <xacro:property name="L3_1" value="SA036__MoJo" />
-  <xacro:property name="L3_2" value="SA046__MoJo" />
-  <xacro:property name="L3_3" value="SA038__MoJo" />
-  <xacro:property name="L4_1" value="SA022__MoJo" />
-  <xacro:property name="L4_2" value="SA050__MoJo" />
-  <xacro:property name="L4_3" value="SA031__MoJo" />
-  <xacro:property name="L5_1" value="SA002__MoJo" />
-  <xacro:property name="L5_2" value="SA003__MoJo" />
-  <xacro:property name="L5_3" value="SA048__MoJo" />
-  <xacro:property name="L6_1" value="SA043__MoJo" />
-  <xacro:property name="L6_2" value="SA005__MoJo" />
-  <xacro:property name="L6_3" value="SA001__MoJo" />
-  <xacro:property name="width" value=".185" />
-  <xacro:property name="length" value=".3" />
-  <xacro:property name="height" value=".0762" />
-  <xacro:property name="leg_y_offset" value=".125" />
-  <link name="kdl_dummy_root" />
-  <joint name="kdl_dummy_root_to_base" type="fixed">
-    <parent link="kdl_dummy_root"/>
-    <child link="base"/>
-  </joint>
-  <!-- base body -->
-  <link name="base">
-    <visual>
-      <origin xyz="0 0 ${height/2}" rpy="0 0 0" />
-      <geometry>
-        <box size="${width} ${length} ${height}" />
-      </geometry>
-      <xacro:silver_material/>
-    </visual>
-    <collision>
-      <origin xyz="0 0 ${height/2}" rpy="0 0 0" />
-      <geometry>
+	<!-- *************************** XACRO MACROS *************************** -->
+	<xacro:property name="PI" value="3.1415926535897931" />
+	<xacro:property name="M_PI" value="3.1415926535897931" />
+	<!-- load macros for modules -->
+	<xacro:include filename="./module_common.xacro"/>
+	<xacro:include filename="./rotary_module.xacro"/>
+	<xacro:include filename="./extension_module.xacro"/>
+	<xacro:include filename="./elbow_module_snake_monster.xacro"/>
+	<xacro:include filename="./leg.xacro"/>
+	<!-- ************************* ROBOT DEFINITION ************************* -->
+	<xacro:property name="L1_1" value="SA014__MoJo" />
+	<xacro:property name="L1_2" value="SA013__MoJo" />
+	<xacro:property name="L1_3" value="SA023__MoJo" />
+	<xacro:property name="L2_1" value="SA037__MoJo" />
+	<xacro:property name="L2_2" value="SA049__MoJo" />
+	<xacro:property name="L2_3" value="SA030__MoJo" />
+	<xacro:property name="L3_1" value="SA036__MoJo" />
+	<xacro:property name="L3_2" value="SA046__MoJo" />
+	<xacro:property name="L3_3" value="SA038__MoJo" />
+	<xacro:property name="L4_1" value="SA022__MoJo" />
+	<xacro:property name="L4_2" value="SA050__MoJo" />
+	<xacro:property name="L4_3" value="SA031__MoJo" />
+	<xacro:property name="L5_1" value="SA002__MoJo" />
+	<xacro:property name="L5_2" value="SA003__MoJo" />
+	<xacro:property name="L5_3" value="SA048__MoJo" />
+	<xacro:property name="L6_1" value="SA043__MoJo" />
+	<xacro:property name="L6_2" value="SA005__MoJo" />
+	<xacro:property name="L6_3" value="SA001__MoJo" />
+	<xacro:property name="width" value=".185" />
+	<xacro:property name="length" value=".3" />
+	<xacro:property name="height" value=".0762" />
+	<xacro:property name="leg_y_offset" value=".125" />
+	<!--link name="kdl_dummy_root" />
+	<joint name="kdl_dummy_root_to_base" type="fixed">
+		<parent link="kdl_dummy_root"/>
+		<child link="base"/>
+	</joint-->
+	<!-- base body -->
+	<link name="base">
+		<visual>
+			<origin xyz="0 0 ${height/2}" rpy="0 0 0" />
+			<geometry>
+				<box size="${width} ${length} ${height}" />
+			</geometry>
+			<xacro:silver_material/>
+		</visual>
+		<collision>
+			<origin xyz="0 0 ${height/2}" rpy="0 0 0" />
+			<geometry>
 	<box size="${width} ${length} ${height}" />
-      </geometry>
-    </collision>
-    <inertial>
-      <origin xyz="0 0 ${height/2}" rpy="0 0 0" />
-      <mass value="1.0"/>
-      <inertia ixx="${1.0/12.0*(length**2+height**2)}" iyy="${1.0/12.0*(width**2+height**2)}" izz="${1.0/12.0*(width**2+length**2)}" ixy="0" ixz="0" iyz="0" />
-    </inertial>
-  </link>
+			</geometry>
+		</collision>
+		<inertial>
+			<origin xyz="0 0 ${height/2}" rpy="0 0 0" />
+			<mass value="1.0"/>
+			<inertia ixx="${1.0/12.0*(length**2+height**2)}" iyy="${1.0/12.0*(width**2+height**2)}" izz="${1.0/12.0*(width**2+length**2)}" ixy="0" ixz="0" iyz="0" />
+		</inertial>
+	</link>
   <link name="xrot">
    <visual>
@@ -119,35 +119,35 @@
       </actuator>
     </transmission>
-  <!-- leg outputs on the base -->
-  <joint name="leg1__OUTPUT_INTERFACE" type="fixed">
-    <parent link="base"/>
-    <child link="${L1_1}__INPUT_INTERFACE"/>
-    <origin xyz="${width/2} ${leg_y_offset} ${height/2}" rpy="-${PI/2} 0 -${PI/2}"/>
-  </joint>
-  <joint name="leg2__OUTPUT_INTERFACE" type="fixed">
-    <parent link="base"/>
-    <child link="${L2_1}__INPUT_INTERFACE"/>
-    <origin xyz="${width/2} 0 ${height/2}" rpy="-${PI/2} 0 -${PI/2}"/>
-  </joint>
-  <joint name="leg3__OUTPUT_INTERFACE" type="fixed">
-    <parent link="base"/>
-    <child link="${L3_1}__INPUT_INTERFACE"/>
-    <origin xyz="${width/2} -${leg_y_offset} ${height/2}" rpy="-${PI/2} 0 -${PI/2}"/>
-  </joint>
-  <joint name="leg6__OUTPUT_INTERFACE" type="fixed">
-    <parent link="base"/>
-    <child link="${L6_1}__INPUT_INTERFACE"/>
-    <origin xyz="${-width/2} ${leg_y_offset} ${height/2}" rpy="-${PI/2} 0 ${PI/2}"/>
-  </joint>
-  <joint name="leg5__OUTPUT_INTERFACE" type="fixed">
-    <parent link="base"/>
-    <child link="${L5_1}__INPUT_INTERFACE"/>
-    <origin xyz="${-width/2} 0 ${height/2}" rpy="-${PI/2} 0 ${PI/2}"/>
-  </joint>
-  <joint name="leg4__OUTPUT_INTERFACE" type="fixed">
-    <parent link="base"/>
-    <child link="${L4_1}__INPUT_INTERFACE"/>
-    <origin xyz="${-width/2} -${leg_y_offset} ${height/2}" rpy="-${PI/2} 0 ${PI/2}"/>
-  </joint>
+	<!-- leg outputs on the base -->
+	<joint name="leg1__OUTPUT_INTERFACE" type="fixed">
+		<parent link="base"/>
+		<child link="${L1_1}__INPUT_INTERFACE"/>
+		<origin xyz="${width/2} ${leg_y_offset} ${height/2}" rpy="-${PI/2} 0 -${PI/2}"/>
+	</joint>
+	<joint name="leg2__OUTPUT_INTERFACE" type="fixed">
+		<parent link="base"/>
+		<child link="${L2_1}__INPUT_INTERFACE"/>
+		<origin xyz="${width/2} 0 ${height/2}" rpy="-${PI/2} 0 -${PI/2}"/>
+	</joint>
+	<joint name="leg3__OUTPUT_INTERFACE" type="fixed">
+		<parent link="base"/>
+		<child link="${L3_1}__INPUT_INTERFACE"/>
+		<origin xyz="${width/2} -${leg_y_offset} ${height/2}" rpy="-${PI/2} 0 -${PI/2}"/>
+	</joint>
+	<joint name="leg6__OUTPUT_INTERFACE" type="fixed">
+		<parent link="base"/>
+		<child link="${L6_1}__INPUT_INTERFACE"/>
+		<origin xyz="${-width/2} ${leg_y_offset} ${height/2}" rpy="-${PI/2} 0 ${PI/2}"/>
+	</joint>
+	<joint name="leg5__OUTPUT_INTERFACE" type="fixed">
+		<parent link="base"/>
+		<child link="${L5_1}__INPUT_INTERFACE"/>
+		<origin xyz="${-width/2} 0 ${height/2}" rpy="-${PI/2} 0 ${PI/2}"/>
+	</joint>
+	<joint name="leg4__OUTPUT_INTERFACE" type="fixed">
+		<parent link="base"/>
+		<child link="${L4_1}__INPUT_INTERFACE"/>
+		<origin xyz="${-width/2} -${leg_y_offset} ${height/2}" rpy="-${PI/2} 0 ${PI/2}"/>
+	</joint>
  <xacro:include filename="$(find kobuki_description)/urdf/sensors/lidar_sensor.urdf.xacro" />
  <xacro:lidar_sensor
@@ -196,10 +196,23 @@
     </inertial>
   </link>
-  <!-- legs -->
-  <xacro:leg leg="leg1" mod1="${L1_1}" mod2="${L1_2}" mod3="${L1_3}"/>
-  <xacro:leg leg="leg2" mod1="${L2_1}" mod2="${L2_2}" mod3="${L2_3}"/>
-  <xacro:leg leg="leg3" mod1="${L3_1}" mod2="${L3_2}" mod3="${L3_3}"/>s
-  <xacro:leg leg="leg4" mod1="${L4_1}" mod2="${L4_2}" mod3="${L4_3}"/>
-  <xacro:leg leg="leg5" mod1="${L5_1}" mod2="${L5_2}" mod3="${L5_3}"/>
-  <xacro:leg leg="leg6" mod1="${L6_1}" mod2="${L6_2}" mod3="${L6_3}"/>
+	<!-- Import all Gazebo-customization elements -->
+	<xacro:include filename="./my_snake_monster.gazebo" />
+	<!-- legs -->
+	<xacro:leg leg="leg1" mod1="${L1_1}" mod2="${L1_2}" mod3="${L1_3}"/>
+	<xacro:leg leg="leg2" mod1="${L2_1}" mod2="${L2_2}" mod3="${L2_3}"/>
+	<xacro:leg leg="leg3" mod1="${L3_1}" mod2="${L3_2}" mod3="${L3_3}"/>
+	<xacro:leg leg="leg4" mod1="${L4_1}" mod2="${L4_2}" mod3="${L4_3}"/>
+	<xacro:leg leg="leg5" mod1="${L5_1}" mod2="${L5_2}" mod3="${L5_3}"/>
+	<xacro:leg leg="leg6" mod1="${L6_1}" mod2="${L6_2}" mod3="${L6_3}"/>
+	 <gazebo>
+		<plugin name="p3d" filename="libgazebo_ros_p3d.so">
+        	<alwaysOn>true</alwaysOn>
+          	<updateRate>1000.0</updateRate>
+          	<bodyName>base</bodyName>
+          	<topicName>nav_msgs</topicName>
+          	<frameName>world</frameName>
+          	<xyzOffsets>0 0 0.0</xyzOffsets>
+          	<rpyOffsets>0 0 0.0</rpyOffsets>
+    	</plugin>
+    </gazebo>
 </robot>

Commit message: Moved the robot

File: gym_gazebo/envs/installation/catkin_ws/src/snakemonster/snake_monster/urdf/my_snake_monster.xacro (robot description, xacro)
@@ -37,5 +37,5 @@
 		<parent link="kdl_dummy_root"/>
 		<child link="base"/>
-	</joint-->
+	</joint -->
 	<!-- base body -->
 	<link name="base">
@@ -197,5 +197,5 @@
   </link>
 	<!-- Import all Gazebo-customization elements -->
-	<xacro:include filename="./my_snake_monster.gazebo" />
+	<!--xacro:include filename="./my_snake_monster.gazebo" /-->
 	<!-- legs -->
 	<xacro:leg leg="leg1" mod1="${L1_1}" mod2="${L1_2}" mod3="${L1_3}"/>
@@ -214,5 +214,5 @@
           	<xyzOffsets>0 0 0.0</xyzOffsets>
           	<rpyOffsets>0 0 0.0</rpyOffsets>
-    	</plugin>
-    </gazebo>
+    		</plugin>
+    	</gazebo>
 </robot>

Commit message: Working code for one joint and also URDF param set

File: gym_gazebo/envs/installation/catkin_ws/src/snakemonster/snake_monster/urdf/my_snake_monster.xacro (robot description, xacro)
@@ -33,9 +33,4 @@
 	<xacro:property name="height" value=".0762" />
 	<xacro:property name="leg_y_offset" value=".125" />
-	<!--link name="kdl_dummy_root" />
-	<joint name="kdl_dummy_root_to_base" type="fixed">
-		<parent link="kdl_dummy_root"/>
-		<child link="base"/>
-	</joint -->
 	<!-- base body -->
 	<link name="base">
@@ -50,5 +45,5 @@
 			<origin xyz="0 0 ${height/2}" rpy="0 0 0" />
 			<geometry>
-	<box size="${width} ${length} ${height}" />
+			<box size="${width} ${length} ${height}" />
 			</geometry>
 		</collision>
@@ -65,5 +60,5 @@
 		<box size="0.02 0.02 0.02"/>
 	</geometry>
-   </visual>
+   	</visual>
     <inertial>
       <mass value="1e-3" />
@@ -76,30 +71,30 @@
     <origin xyz="0 0 0.0762" rpy="0 0 0"/>
     <axis xyz="1 0 0"/>
-      <dynamics damping=".05" friction="0.2"/>
-      <limit effort="100.0" lower="-1.57" upper="1.57" velocity="2.208932"/>
+    <dynamics damping=".05" friction="0.2"/>
+    <limit effort="100.0" lower="-1.57" upper="1.57" velocity="2.208932"/>
  </joint>
 <transmission name="xrot_trans">
-      <type>transmission_interface/SimpleTransmission</type>
-      <joint name="xrot_joint">
-	<hardwareInterface>EffortJointInterface</hardwareInterface>
-      </joint>
-      <actuator name="xrot_motor">
-	<hardwareInterface>EffortJointInterface</hardwareInterface>
-	<mechanicalReduction>300</mechanicalReduction>
-      </actuator>
+    <type>transmission_interface/SimpleTransmission</type>
+    <joint name="xrot_joint">
+		<hardwareInterface>EffortJointInterface</hardwareInterface>
+    </joint>
+    <actuator name="xrot_motor">
+		<hardwareInterface>EffortJointInterface</hardwareInterface>
+		<mechanicalReduction>300</mechanicalReduction>
+    </actuator>
     </transmission>
-  <link name="yrot">
-   <visual>
-	<origin xyz="0 0 0.01" rpy="0 0 0" />
-	<geometry>
-		<box size="0.02 0.02 0.02"/>
-	</geometry>
-   </visual>
+<link name="yrot">
+	<visual>
+		<origin xyz="0 0 0.01" rpy="0 0 0" />
+		<geometry>
+			<box size="0.02 0.02 0.02"/>
+		</geometry>
+	</visual>
     <inertial>
       <mass value="1e-3" />
       <inertia ixx="1e-3" ixy="0" ixz="0" iyy="1e-3" iyz="0" izz="1e-3" />
     </inertial>
-  </link>
- <joint name="yrot_joint" type="revolute">
+</link>
+<joint name="yrot_joint" type="revolute">
     <parent link="xrot"/>
     <child link="yrot"/>
@@ -108,15 +103,15 @@
       <dynamics damping=".05" friction="0.2"/>
       <limit effort="7.0" lower="-1.57" upper="1.57" velocity="2.208932"/>
- </joint>
+</joint>
 <transmission name="yrot_trans">
-      <type>transmission_interface/SimpleTransmission</type>
-      <joint name="yrot_joint">
-	<hardwareInterface>EffortJointInterface</hardwareInterface>
-      </joint>
-      <actuator name="yrot_motor">
-	<hardwareInterface>EffortJointInterface</hardwareInterface>
-	<mechanicalReduction>300</mechanicalReduction>
-      </actuator>
-    </transmission>
+    <type>transmission_interface/SimpleTransmission</type>
+    <joint name="yrot_joint">
+		<hardwareInterface>EffortJointInterface</hardwareInterface>
+    </joint>
+    <actuator name="yrot_motor">
+		<hardwareInterface>EffortJointInterface</hardwareInterface>
+		<mechanicalReduction>300</mechanicalReduction>
+    </actuator>
+</transmission>
 	<!-- leg outputs on the base -->
 	<joint name="leg1__OUTPUT_INTERFACE" type="fixed">
@@ -150,21 +145,6 @@
 		<origin xyz="${-width/2} -${leg_y_offset} ${height/2}" rpy="-${PI/2} 0 ${PI/2}"/>
 	</joint>
- <!--xacro:include filename="$(find kobuki_description)/urdf/sensors/lidar_sensor.urdf.xacro" />
- <xacro:lidar_sensor
-    name="sonar2"
-    parent="yrot"
-    ros_topic="sonar_front"
-    update_rate="10"
-    min_range="0.06"
-    max_range="4.0"
-    field_of_view_horizontal="${270*M_PI/180}"
-    field_of_view_vertical="${1*M_PI/180}"
-    ray_count_horizontal="200"
-    ray_count_vertical="1"
-    sensor_mesh="lidar_lite_v2_withRay/meshes/lidar_lite_v2_withRay.dae">
-    <origin xyz="0 0 0.405" rpy="0 0 1.57"/>
-  </xacro:lidar_sensor-->
-  <!-- Import all Gazebo-customization elements -->
-  <xacro:include filename="./my_snake_monster.gazebo" />
+<!-- Import all Gazebo-customization elements -->
+<xacro:include filename="./my_snake_monster.gazebo" />
 <xacro:property name="camera_link" value="0.05"/><!-- Size of square 'camera' box --><joint name="camera_joint" type="fixed"><axis xyz="0 1 0"/><origin xyz="0 0.125 0.052" rpy="0 0 1.57"/><parent link="base"/><child link="camera_link"/></joint><!-- Camera --><link name="camera_link"><collision><origin xyz="0 0 0.052" rpy="0 0 1.57"/><geometry><box size="${camera_link} ${camera_link} ${camera_link}"/></geometry></collision><visual><origin xyz="-0.02 -0.02 0.024" rpy="0 0 0"/><geometry><mesh filename="package://snake_monster/meshes/gopro.dae"/></geometry><material name="red"/></visual><inertial><mass value="1e-5"/><origin xyz="0 0 0" rpy="0 0 0"/><inertia ixx="1e-6" ixy="0" ixz="0" iyy="1e-6" iyz="0" izz="1e-6"/></inertial></link>
    <xacro:property name="imu_link" value="0.05" /> <!-- Size of square 'camera' box -->
@@ -180,5 +160,5 @@
       <origin xyz="0 0 0.052" rpy="0 0 1.57"/>
       <geometry>
-    <box size="0.1 0.1 0.1"/>
+    		<box size="0.1 0.1 0.1"/>
       </geometry>
     </collision>
@@ -186,5 +166,5 @@
       <origin xyz="-0.02 -0.02 0.024" rpy="0 0 0"/>
       <geometry>
-    <box size ="0.1 0.1 0.1"/>
+    		<box size ="0.1 0.1 0.1"/>
       </geometry>
       <material name="red"/>
@@ -197,5 +177,4 @@
   </link>
 	<!-- Import all Gazebo-customization elements -->
-	<!--xacro:include filename="./my_snake_monster.gazebo" /-->
 	<!-- legs -->
 	<xacro:leg leg="leg1" mod1="${L1_1}" mod2="${L1_2}" mod3="${L1_3}"/>
@@ -205,5 +184,5 @@
 	<xacro:leg leg="leg5" mod1="${L5_1}" mod2="${L5_2}" mod3="${L5_3}"/>
 	<xacro:leg leg="leg6" mod1="${L6_1}" mod2="${L6_2}" mod3="${L6_3}"/>
-	 <gazebo>
+	<gazebo>
 		<plugin name="p3d" filename="libgazebo_ros_p3d.so">
         	<alwaysOn>true</alwaysOn>
@@ -214,5 +193,5 @@
           	<xyzOffsets>0 0 0.0</xyzOffsets>
           	<rpyOffsets>0 0 0.0</rpyOffsets>
-    		</plugin>
-    	</gazebo>
+    	</plugin>
+    </gazebo>
 </robot>

Commit message: Adding reward bug fixes

File: gym_gazebo/envs/installation/catkin_ws/src/snakemonster/snake_monster/urdf/my_snake_monster.xacro (robot description, xacro)
@@ -160,5 +160,5 @@
       <origin xyz="0 0 0.052" rpy="0 0 1.57"/>
       <geometry>
-    		<box size="0.1 0.1 0.1"/>
+    		<box size="0.01 0.01 0.01"/>
       </geometry>
     </collision>
